File: mister-vector/mister-vector.kicad_sch (KiCad schematic)
At the start: 132 parts, among them IC1 SN74ALVCH16841DL, IC2 7432D, IC3 74139D, IC4 SN74ALVCH16841DL, IC5 TL084, IC6 SN74ALVCH16841DL, IC7 TL084, J1 618015330923, J2 AUDIO_JACK_3.5MM_KIT, J3 618015330923, U1 VASD1-SIP

Commit message: reworking for r2r-dac and edge triggered buffers
Parts:
- removed C1, C13: 100nF, mister-vector:C0603, symbol mister-vector-eagle-import:C-EUC0603
- removed C14, C17, C18, C6, C7: 4.7uF, mister-vector:CT3528, symbol mister-vector-eagle-import:CPOL-EUCT3528
- removed C15, C16, C19, C20: 0.1uF, mister-vector:C0603, symbol mister-vector-eagle-import:C-USC0603
- removed IC1, IC4, IC6: SN74ALVCH16841DL, mister-vector:SOP50P810X120-56N, symbol mister-vector-eagle-import:SN74ALVCH16841DL
- removed IC2: 7432D, mister-vector:SO14, symbol mister-vector-eagle-import:7432D
- removed IC3: 74139D, mister-vector:SO16, symbol mister-vector-eagle-import:74139D
- removed J1, J3: 618015330923, mister-vector:618015330923, symbol mister-vector-eagle-import:618015330923
- removed JP1: JP2E, mister-vector:JP2, symbol mister-vector-eagle-import:JP2E
- removed R1, R2, R3, R30, R31, R32, R60, R61, R77, R78: 510R, mister-vector:R0603, symbol mister-vector-eagle-import:R-EU_R0603
- removed R10, R38, R39, R40, R66, R67, R8, R9: 2K2, mister-vector:R0603, symbol mister-vector-eagle-import:R-EU_R0603
- removed R11, R25, R29, R7: 100R, mister-vector:R0603, symbol mister-vector-eagle-import:R-EU_R0603
- removed R12, R13, R14, R43, R44, R45, R71, R72: 4K3, mister-vector:R0603, symbol mister-vector-eagle-import:R-EU_R0603
- removed R15, R16, R17, R48, R49, R50, R73, R74: 9K1, mister-vector:R0603, symbol mister-vector-eagle-import:R-EU_R0603
- removed R18, R19, R20, R51, R52, R53, R75, R76: 18K, mister-vector:R0603, symbol mister-vector-eagle-import:R-EU_R0603
- removed R21, R24, R26: 10K, mister-vector:R0603, symbol mister-vector-eagle-import:R-US_R0603
- removed R33, R34, R35, R4, R5, R6, R62, R63: 1K1, mister-vector:R0603, symbol mister-vector-eagle-import:R-EU_R0603
- removed R79, R80: 36K, mister-vector:R0603, symbol mister-vector-eagle-import:R-EU_R0603
- removed R83, R84: 75K, mister-vector:R0603, symbol mister-vector-eagle-import:R-EU_R0603
- removed R85, R86: 150K, mister-vector:R0603, symbol mister-vector-eagle-import:R-EU_R0603
- removed R90, R91: 300K, mister-vector:R0603, symbol mister-vector-eagle-import:R-EU_R0603
- added C14, C17, C18: 4.7uF, Capacitor_SMD:C_0805_2012Metric, symbol Device:C_Small_US
- added C15, C19: 100nF, Capacitor_SMD:C_0402_1005Metric, symbol mister-vector-eagle-import:C-EUC0603
- added C21, C22, C23, C24: 100nF, Capacitor_SMD:C_0402_1005Metric, symbol Device:C
- added C6, C7: 4.7uF BP, Capacitor_SMD:C_0805_2012Metric, symbol Device:C
- added U2, U3, U4: SN74LVC821ADGVR, Package_SO:SOIC-24W_7.5x15.4mm_P1.27mm, symbol SN74LVC821ADGVR:SN74LVC821ADGVR
- C10, C2, C3, C4, C5, C8, C9: footprint mister-vector:C0603 -> Capacitor_SMD:C_0402_1005Metric
Connections:
- net +5V: now also C17.1
- net GND: now also C10.1, C9.2, C14.2, C15.2, C17.2, C18.2, C19.1, C21.1, C22.1, C23.1, C24.1, U2.1 (*OE), U2.12 (GND), U3.1 (*OE), U3.12 (GND), U4.1 (*OE), U4.12 (GND); no longer C10.2, C9.1
- net at C5.2, R23.2: now also C6.1
- net at R27.2, R28.1: now also C9.1; no longer C9.2
- net at R28.2: now also C10.2, C7.1; no longer C10.1
- net at J2.RING: now also C6.2
- net at J2.TIP: now also C7.2
- net +12V_OPAMP renamed +12V
- net +12V: now also C14.1, C15.1, C21.2, C23.2
- net +3V3 renamed +3.3V
- net +3.3V: now also U2.24 (VCC), U3.24 (VCC), U4.24 (VCC)
- net -12V_OPAMP renamed -12V
- net -12V: now also C18.1, C19.2, C22.2, C24.2
- net B+ renamed B
- net G+ renamed G
- net HSYNC: no longer names the net of GPIO1.20
- net R+ renamed R
- net SD_CLK renamed CLK_RGB
- net CLK_RGB: now also U4.13 (CLK)
- net SD_DAT0 renamed CLK_Y
- net CLK_Y: now also U3.13 (CLK)
- net SD_DAT1 renamed CLK_X
- net CLK_X: now also U2.13 (CLK)
- net VEC_X+ renamed VEC_X
- net VEC_Y+ renamed VEC_Y
- net VGA2_B renamed DAC_B
- net VGA2_G renamed DAC_G
- net VGA2_R renamed DAC_R
- net VGA_B0: no longer names the net of GPIO1.22
- net VGA_B1: no longer names the net of GPIO1.24
- net VGA_B2: no longer names the net of GPIO1.26
- net VGA_B3 renamed D6
- net D6: now also U2.8 (7D), U3.8 (7D), U4.8 (7D)
- net VGA_B4 renamed D7
- net D7: now also U2.9 (8D), U3.9 (8D), U4.9 (8D)
- net VGA_B5 renamed D8
- net D8: now also U2.10 (9D), U3.10 (9D), U4.10 (9D)
- net VGA_G0 renamed D0
- net D0: now also U2.2 (1D), U3.2 (1D), U4.2 (1D)
- net VGA_G1 renamed D1
- net D1: now also U2.3 (2D), U3.3 (2D), U4.3 (2D)
- net VGA_G2 renamed D2
- net D2: now also U2.4 (3D), U3.4 (3D), U4.4 (3D)
- net VGA_G3 renamed D3
- net D3: now also U2.5 (4D), U3.5 (4D), U4.5 (4D)
- net VGA_G4 renamed D4
- net D4: now also U2.6 (5D), U3.6 (5D), U4.6 (5D)
- net VGA_G5 renamed D5
- net D5: now also U2.7 (6D), U3.7 (6D), U4.7 (6D)
- net VGA_R0: no longer names the net of GPIO1.40
- net VGA_R1: no longer names the net of GPIO1.38
- net VGA_R2: no longer names the net of GPIO1.36
- net VGA_R3: no longer names the net of GPIO1.34
- net VGA_R4: no longer names the net of GPIO1.32
- net VGA_R5: no longer names the net of GPIO1.28
- net VSYNC renamed D9
- net D9: now also U2.11 (10D), U3.11 (10D), U4.11 (10D)
- new net R2R_DAC_B/D0: U4.17 (7Q)
- new net R2R_DAC_B/D1: U4.16 (8Q)
- new net R2R_DAC_B/D2: U4.15 (9Q)
- new net R2R_DAC_G/D0: U4.20 (4Q)
- new net R2R_DAC_G/D1: U4.19 (5Q)
- new net R2R_DAC_G/D2: U4.18 (6Q)
- new net R2R_DAC_R/D0: U4.23 (1Q)
- new net R2R_DAC_R/D1: U4.22 (2Q)
- new net R2R_DAC_R/D2: U4.21 (3Q)
- new net R2R_DAC_X/D0: U2.23 (1Q)
- new net R2R_DAC_X/D1: U2.22 (2Q)
- new net R2R_DAC_X/D2: U2.21 (3Q)
- new net R2R_DAC_X/D3: U2.20 (4Q)
- new net R2R_DAC_X/D4: U2.19 (5Q)
- new net R2R_DAC_X/D5: U2.18 (6Q)
- new net R2R_DAC_X/D6: U2.17 (7Q)
- new net R2R_DAC_X/D7: U2.16 (8Q)
- new net R2R_DAC_X/D8: U2.15 (9Q)
- new net R2R_DAC_X/D9: U2.14 (10Q)
- new net R2R_DAC_Y/D0: U3.23 (1Q)
- new net R2R_DAC_Y/D1: U3.22 (2Q)
- new net R2R_DAC_Y/D2: U3.21 (3Q)
- new net R2R_DAC_Y/D3: U3.20 (4Q)
- new net R2R_DAC_Y/D4: U3.19 (5Q)
- new net R2R_DAC_Y/D5: U3.18 (6Q)
- new net R2R_DAC_Y/D6: U3.17 (7Q)
- new net R2R_DAC_Y/D7: U3.16 (8Q)
- new net R2R_DAC_Y/D8: U3.15 (9Q)
- new net R2R_DAC_Y/D9: U3.14 (10Q)
Other:
- added sheet R2R_DAC_B (r2rdac3.kicad_sch)
- added sheet R2R_DAC_G (r2rdac3.kicad_sch)
- added sheet R2R_DAC_R (r2rdac3.kicad_sch)
- added sheet R2R_DAC_X (r2rdac10.kicad_sch)
- added sheet R2R_DAC_Y (r2rdac10.kicad_sch)
- note added: "DE10-Nano 2x40 connector"
- note added: "non transparent edge trigger latch"
- note removed: "3V3"
- note removed: "5V"
- note removed: "<- ~{VGA_EN}"
- note removed: "When DACx_LAT is High, the latches are in passthrough. When DACx_LAT goes Low, the data gets latched."
- moved on the sheet: C11, C12, C2, C3, GPIO1, IC5A, IC5B, IC5C, IC5D, IC7A, IC7B, IC7C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

Commit message: hierarchical schematic, add libraries
Parts:
- removed C10, C4, C5, C9: 10nF, Capacitor_SMD:C_0402_1005Metric, symbol mister-vector-eagle-import:C-EUC0603
- removed C11, C12: 1.0uF, mister-vector:C0603, symbol mister-vector-eagle-import:C-USC0603
- removed C2, C3, C8: 100nF, Capacitor_SMD:C_0402_1005Metric, symbol mister-vector-eagle-import:C-EUC0603
- removed C21, C22, C23, C24: 100nF, Capacitor_SMD:C_0402_1005Metric, symbol Device:C
- removed C6, C7: 4.7uF BP, Capacitor_SMD:C_0805_2012Metric, symbol Device:C
- removed IC5, IC7: TL084, mister-vector:SOIC-14, symbol mister-vector-eagle-import:TL084
- removed J2: AUDIO_JACK_3.5MM_KIT, mister-vector:AUDIO-JACK-KIT, symbol mister-vector-eagle-import:AUDIO_JACK_3.5MM_KIT
- removed OFFSET0, X_SIZE0, Y_SIZE0: 20K, mister-vector:B25P, symbol mister-vector-eagle-import:TRIM_EU-B25P
- removed R22, R23, R27, R28: 510R, mister-vector:R0603, symbol mister-vector-eagle-import:R-EU_R0603
- removed R36, R37, R54, R55, R64, R65, R81, R82: 75R, mister-vector:R0603, symbol mister-vector-eagle-import:R-US_R0603
- removed R41, R42, R56, R57, R68, R69, R70, R87, R88, R89: 10K, mister-vector:R0603, symbol mister-vector-eagle-import:R-US_R0603
- removed R46, R47, R58, R59: 4K7, mister-vector:R0603, symbol mister-vector-eagle-import:R-US_R0603
- removed U$1, U$2, U$3, U$4: PLATED_HOLE3.6MM, mister-vector:PLATED_HOLE_3.6MM, symbol mister-vector-eagle-import:PLATED_HOLE3.6MM
- removed U1: VASD1-SIP, mister-vector:NMA, symbol mister-vector-eagle-import:NMA
- removed U2, U3, U4: SN74LVC821ADGVR, Package_SO:SOIC-24W_7.5x15.4mm_P1.27mm, symbol SN74LVC821ADGVR:SN74LVC821ADGVR
- removed VEC_OUT1: 22-23-2071, mister-vector:22-23-2071, symbol mister-vector-eagle-import:22-23-2071
- added H1, H2, H3, H4: MountingHole_Pad, MountingHole:MountingHole_3mm_Pad_Via, symbol Mechanical:MountingHole_Pad
- added H5: FAN1, MountingHole:MountingHole_3mm, symbol Mechanical:MountingHole_Pad
- added H6: FAN2, MountingHole:MountingHole_3mm, symbol Mechanical:MountingHole_Pad
- added H7: FAN3, MountingHole:MountingHole_3mm, symbol Mechanical:MountingHole_Pad
- added H8: FAN4, MountingHole:MountingHole_3mm, symbol Mechanical:MountingHole_Pad
- added J10: DC-005-2.5A-2.0 C319099, Connector_BarrelJack:BarrelJack_Horizontal, symbol Connector:Barrel_Jack_Switch
- added J100: FAN, Connector_PinHeader_2.54mm:PinHeader_1x03_P2.54mm_Vertical, symbol Connector_Generic:Conn_01x03
- added J8: Jamma_con, Jamma:JAMMA-56, symbol Jamma:Jamma_con
- added R57, R58: 0, Resistor_SMD:R_0402_1005Metric, symbol Device:R_Small_US
- added U1: RD-0512D, RD-0512D:CONV_RD-0512D, symbol RD-0512D:RD-0512D
- C1: renamed from C15; LCSC (none) -> C307331
- C2: renamed from C14; LCSC (none) -> C1779
- C3: renamed from C17; LCSC (none) -> C1779
- C4: renamed from C19; LCSC (none) -> C307331
- C5: renamed from C18; LCSC (none) -> C1779
- renumbered GPIO1 to J7
Connections:
- net +12V: now also U1.6 (+VOUT)
- net +3.3V: now also R57.1; no longer J7.29
- net +5V: now also J10.1, J100.2 (Pin_2), J8.3 (+5V), J8.4 (+5V), J8.C (+5V), J8.D (+5V), R58.1, U1.1 (+VIN); no longer J7.11
- net -12V: now also U1.4 (-VOUT)
- net CLK_RGB: now also J7.26; no longer J7.14
- net CLK_X: now also J7.22; no longer J7.18
- net CLK_Y: now also J7.24; no longer J7.16
- net D0: now also J7.32; no longer J7.39
- net D1: now also J7.34; no longer J7.37
- net D2: now also J7.36; no longer J7.35
- net D3: now also J7.38; no longer J7.33
- net D4: now also J7.40; no longer J7.31
- net D5: now also J7.39; no longer J7.27
- net D6: now also J7.37; no longer J7.25
- net D7: now also J7.35; no longer J7.23
- net D8: now also J7.33; no longer J7.21
- net D9: now also J7.31; no longer J7.19
- net GND: now also H1.1, H2.1, H3.1, H4.1, H5.1, H6.1, H7.1, H8.1, J10.2, J10.3, J100.1 (Pin_1), J8.1 (GND), J8.14 (VIDEO_GND), J8.2 (GND), J8.27 (GND), J8.28 (GND), J8.A (GND), J8.B (GND), J8.e (GND), J8.f (GND), U1.2 (-VIN), U1.5 (COM)
- net CLK_P21: now reaches J7.20
- new net: J7.11, R58.2
- new net: J7.29, R57.2
- new net +12V_NC: J8.6 (+12V), J8.F (+12V)
- new net -5V_NC: J8.5 (-5V), J8.E (-5V)
- new net CLK_P10: J7.14
- new net CLK_P11: J7.18
- new net CLK_P20: J7.16
- new net JAMMA_P1_BUTTON1: J8.22 (P1_BUTTON_1)
- new net JAMMA_P1_BUTTON2: J8.23 (P1_BUTTON_2)
- new net JAMMA_P1_BUTTON3: J8.24 (P1_BUTTON_3)
- new net JAMMA_P1_BUTTON4: J8.25 (P1_BUTTON_4)
- new net JAMMA_P1_COIN: J8.16 (COIN_1)
- new net JAMMA_P1_D: J8.19 (P1_DOWN)
- new net JAMMA_P1_L: J8.20 (P1_LEFT)
- new net JAMMA_P1_R: J8.21 (P1_RIGHT)
- new net JAMMA_P1_START: J8.17 (START_1)
- new net JAMMA_P1_U: J8.18 (P1_UP)
- new net JAMMA_P2_BUTTON1: J8.Z (P2_BUTTON_1)
- new net JAMMA_P2_BUTTON2: J8.a (P2_BUTTON_2)
- new net JAMMA_P2_BUTTON3: J8.b (P2_BUTTON_3)
- new net JAMMA_P2_BUTTON4: J8.c (P2_BUTTON_4)
- new net JAMMA_P2_COIN: J8.T (COIN_2)
- new net JAMMA_P2_D: J8.W (P2_DOWN)
- new net JAMMA_P2_L: J8.X (P2_LEFT)
- new net JAMMA_P2_R: J8.Y (P2_RIGHT)
- new net JAMMA_P2_START: J8.U (START_2)
- new net JAMMA_P2_U: J8.V (P2_UP)
- new net JAMMA_PIN_11(Y): J8.11 (AUDIO+)
- new net JAMMA_PIN_M(X): J8.M (TEST)
- new net JAMMA_SERVICE: J8.R (SERVICE)
- new net JAMMA_SPEAKER+: J8.10 (SPEAKER+)
- new net JAMMA_SPEAKER-: J8.L (SPEAKER-)
- new net JAMMA_TEST: J8.15 (COIN_3)
- new net JAMMA_TILT: J8.S (COIN_4)
- new net JAMMA_VIDEO_B: J8.13 (VIDEO_BLUE)
- new net JAMMA_VIDEO_G: J8.N (VIDEO_GREEN)
- new net JAMMA_VIDEO_R: J8.12 (VIDEO_RED)
- new net JAMMA_VIDEO_SYNC: J8.P (VIDEO_SYNC)
- no-connect marks 0 -> 3
Other:
- removed sheet R2R_DAC_B
- removed sheet R2R_DAC_G
- removed sheet R2R_DAC_R
- removed sheet R2R_DAC_X
- removed sheet R2R_DAC_Y
- added sheet Audio (audio.kicad_sch)
- added sheet Input P1 (digital.kicad_sch)
- added sheet Input P2 (digital.kicad_sch)
- added sheet Vector Amplifiers (vector-amps.kicad_sch)
- added sheet Vector DACs (vector-dacs.kicad_sch)
- note added: "/VGA_EN"
- note added: "5V output to DE10"
- note added: "COIN COUNTER1"
- note added: "COIN COUNTER2"
- note added: "COIN LOCKOUT1"
- note added: "COIN LOCKOUT2"
- note added: "DE10-Nano 2x40 GPIO1"
- note added: "GPIO_1[0] PIN_Y15"
- note added: "GPIO_1[10] PIN_AG25"
- note added: "GPIO_1[11] PIN_AH26"
- note added: "GPIO_1[12] PIN_AH24"
- note added: "GPIO_1[13] PIN_AF25"
- note added: "GPIO_1[14] PIN_AG23"
- note added: "GPIO_1[15] PIN_AF23"
- note added: "GPIO_1[16] PIN_AG24"
- note added: "GPIO_1[17] PIN_AH22"
- note added: "GPIO_1[18] PIN_AH21"
- note added: "GPIO_1[19] PIN_AG21"
- note added: "GPIO_1[1] PIN_AC24"
- note added: "GPIO_1[20] PIN_AH23"
- note added: "GPIO_1[21] PIN_AA20"
- note added: "GPIO_1[22] PIN_AF22"
- note added: "GPIO_1[23] PIN_AE22"
- note added: "GPIO_1[24] PIN_AG20"
- note added: "GPIO_1[25] PIN_AF21"
- note added: "GPIO_1[26] PIN_AG19"
- note added: "GPIO_1[27] PIN_AH19"
- note added: "GPIO_1[28] PIN_AG18"
- note added: "GPIO_1[29] PIN_AH18"
- note added: "GPIO_1[2] PIN_AA15"
- note added: "GPIO_1[30] PIN_AF18"
- note added: "GPIO_1[31] PIN_AF20"
- note added: "GPIO_1[32] PIN_AG15"
- note added: "GPIO_1[33] PIN_AE20"
- note added: "GPIO_1[34] PIN_AE19"
- note added: "GPIO_1[35] PIN_AE17"
- note added: "GPIO_1[3] PIN_AD26"
- note added: "GPIO_1[4] PIN_AG28"
- note added: "GPIO_1[5] PIN_AF28"
- note added: "GPIO_1[6] PIN_AE25"
- note added: "GPIO_1[7] PIN_AF27"
- note added: "GPIO_1[8] PIN_AG26"
- note added: "GPIO_1[9] PIN_AH27"
- note added: "KEY"
- note added: "PART SIDE"
- note added: "SOLDER SIDE"
- note added: "arcade switches are open or closed to ground so pull up is internal to this pcb"
- note added: "esd protection read 6 inputs at a time to bus 2 kHz scan and debounce in fpga"
- note added: "we don't use JAMMA 12V to reduce noise we generate our own +/-12V references"
- note removed: "DE10-Nano 2x40 connector"
- note removed: "GPIO_1[0]"
- note removed: "GPIO_1[10]"
- note removed: "GPIO_1[11]"
- note removed: "GPIO_1[12]"
- note removed: "GPIO_1[13]"
- note removed: "GPIO_1[14]"
- note removed: "GPIO_1[15]"
- note removed: "GPIO_1[16]"
- note removed: "GPIO_1[17]"
- note removed: "GPIO_1[18]"
- note removed: "GPIO_1[19]"
- note removed: "GPIO_1[1]"
- note removed: "GPIO_1[20]"
- note removed: "GPIO_1[21]"
- note removed: "GPIO_1[22]"
- note removed: "GPIO_1[23]"
- note removed: "GPIO_1[24]"
- note removed: "GPIO_1[25]"
- note removed: "GPIO_1[26]"
- note removed: "GPIO_1[27]"
- note removed: "GPIO_1[28]"
- note removed: "GPIO_1[29]"
- note removed: "GPIO_1[2]"
- note removed: "GPIO_1[30]"
- note removed: "GPIO_1[31]"
- note removed: "GPIO_1[32]"
- note removed: "GPIO_1[33]"
- note removed: "GPIO_1[34]"
- note removed: "GPIO_1[35]"
- note removed: "GPIO_1[3]"
- note removed: "GPIO_1[4]"
- note removed: "GPIO_1[5]"
- note removed: "GPIO_1[6]"
- note removed: "GPIO_1[7]"
- note removed: "GPIO_1[8]"
- note removed: "GPIO_1[9]"
- note removed: "non transparent edge trigger latch"
- moved on the sheet: C1, C2, C3, C4, C5, J7
